Commit message: correction

File: src/diff_robot_sim_1/diff_robot_description/urdf/diff_robot.xacro (robot description, xacro)
@@ -102,8 +102,8 @@
         <inertial>
             <origin xyz="0.0 0.0 0.0" rpy="0.0 0.0 0.0"/>
-            <mass value="0.1"/>
+            <mass value="1.0"/>
             <inertia ixx="0.0" ixy="0.0" ixz="0.0" iyy="0.0" iyz="0.0" izz="0.0"/>
         </inertial>
-        <visual name="front_caster_virsual">
+        <visual name="front_caster_visual">
             <origin xyz="0.0 0.0 0.0" rpy="0.0 0.0 0.0"/>
             <geometry>
@@ -111,5 +111,5 @@
             </geometry>
             <material name="">
-                <color rgba="1.0 0.0 0.0 1.0"/>
+                <color rgba="1.0 1.0 1.0 1.0"/>
                 <texture filename=""/>
             </material>
@@ -132,8 +132,8 @@
         <inertial>
             <origin xyz="0.0 0.0 0.0" rpy="0.0 0.0 0.0"/>
-            <mass value="0.1"/>
+            <mass value="1.0"/>
             <inertia ixx="0.0" ixy="0.0" ixz="0.0" iyy="0.0" iyz="0.0" izz="0.0"/>
         </inertial>
-        <visual name="back_caster_virsual">
+        <visual name="back_caster_visual">
             <origin xyz="0.0 0.0 0.0" rpy="0.0 0.0 0.0"/>
             <geometry>
@@ -141,5 +141,5 @@
             </geometry>
             <material name="">
-                <color rgba="1.0 0.0 0.0 1.0"/>
+                <color rgba="1.0 1.0 1.0 1.0"/>
                 <texture filename=""/>
             </material>

Commit message: LiDAR_1

File: src/diff_robot_sim_1/diff_robot_description/urdf/diff_robot.xacro (robot description, xacro)
@@ -16,5 +16,5 @@
         <!-- not needed now to change-->
             <origin xyz="0.0 0.0 0.0" rpy="0.0 0.0 0.0"/>
-            <mass value="1.0"/>
+            <mass value="5.0"/>
             <inertia ixx="0.0" ixy="0.0" ixz="0.0" iyy="0.0" iyz="0.0" izz="0.0"/>
         </inertial>
@@ -40,6 +40,6 @@
         <inertial>
             <origin xyz="0.0 0.0 0.0" rpy="0.0 0.0 0.0"/>
-            <mass value="1.0"/>
-            <inertia ixx="0.0" ixy="0.0" ixz="0.0" iyy="0.0" iyz="0.0" izz="0.0"/>
+            <mass value="5.0"/>
+            <inertia ixx="0.1" ixy="0.0" ixz="0.0" iyy="0.1" iyz="0.0" izz="0.1"/>
         </inertial>
         <visual name="left_wheel_visual">
@@ -71,6 +71,6 @@
         <inertial>
             <origin xyz="0.0 0.0 0.0" rpy="0.0 0.0 0.0"/>
-            <mass value="1.0"/>
-            <inertia ixx="0.0" ixy="0.0" ixz="0.0" iyy="0.0" iyz="0.0" izz="0.0"/>
+            <mass value="5.0"/>
+            <inertia ixx="0.1" ixy="0.0" ixz="0.0" iyy="0.1" iyz="0.0" izz="0.1"/>
         </inertial>
         <visual name="right_wheel_visual">
@@ -159,3 +159,38 @@
         <limit lower="0.0" upper="0.0" effort="0.0" velocity="0.0"/>
     </joint>
+    <link name="lidar_link">
+        <inertial>
+            <origin xyz="0.0 0.0 0.0" rpy="0.0 0.0 0.0"/>
+            <mass value="0.1"/>
+            <inertia ixx="0.0" ixy="0.0" ixz="0.0" iyy="0.0" iyz="0.0" izz="0.0"/>
+        </inertial>
+        <visual name="lidar_link_visual">
+            <origin xyz="0.0 0.0 0.0" rpy="0.0 0.0 0.0"/>
+            <geometry>
+                <mesh filename="package://diff_robot_description/meshes/lidar_link.STL"/>
+            </geometry>
+            <material name="">
+                <color rgba="1.0 0.0 0.0 1.0"/>
+                <texture filename=""/>
+            </material>
+        </visual>
+        <collision>
+            <origin xyz="0.0 0.0 0.0" rpy="0.0 0.0 0.0"/>
+            <geometry>
+                <box size="0.1 0.1 0.1"/>
+            </geometry>
+        </collision>
+    </link>
+    <joint name="lidar_joint" type="fixed">
+        <origin xyz="0.11 0.0 0.12" rpy="1.5708 0.0 1.5708"/>
+        <parent link="base_link"/>
+        <child link="lidar_link"/>
+    </joint>
+    <link name="laser_data_link">
+    </link>
+    <joint name="laser_data_joint" type="fixed">
+        <origin xyz="0.0 0.0 0.0" rpy="0.0 -1.5708 -1.5708"/>
+        <parent link="lidar_link"/>
+        <child link="laser_data_link"/>
+    </joint>
 </robot>

Commit message: URDF_ADDED

File: src/diff_robot_sim_1/diff_robot_description/urdf/diff_robot.xacro (robot description, xacro)
@@ -183,5 +183,5 @@
     </link>
     <joint name="lidar_joint" type="fixed">
-        <origin xyz="0.11 0.0 0.12" rpy="1.5708 0.0 1.5708"/>
+        <origin xyz="0.11 0.0 0.12" rpy="1.5708 0.0 0.0"/>
         <parent link="base_link"/>
         <child link="lidar_link"/>
