Commit message: LiDAR_Gazebo_Rviz

File: src/my_robot_descirption_6/urdf/my_robot_descirption_6.xacro (robot description, xacro)
@@ -1,8 +1,13 @@
 <?xml version="1.0" encoding="utf-8"?>
-<!-- This URDF was automatically created by SolidWorks to URDF Exporter! Originally created by Stephen Brawner (brawner@gmail.com)
-     Commit Version: 1.6.0-1-g15f4949  Build Version: 1.6.7594.29634
-     For more information, please see http://wiki.ros.org/sw_urdf_exporter -->
-<robot
-  name="my_robot_descirption_6">
+<robot xmlns:xacro="http://www.ros.org/wiki/xacro" name="my_robot_descirption_6">
+  <xacro:include filename="$(find my_robot_descirption_6)/urdf/my_robot.gazebo"/>
+  <!--dummy robot base-->
+  <link name="robot_footprint">
+  </link>
+  <joint name="robot_footprint_joint" type="fixed">
+    <parent link="robot_footprint"/>
+    <child link="base_link"/>
+    <origin xyz="0.0 0.0 0.0" rpy="0.0 0.0 0.0"/>
+  </joint>
   <link
     name="base_link">
@@ -32,5 +37,5 @@
         name="">
         <color
-          rgba="0.898039215686275 0.917647058823529 0.929411764705882 1" />
+          rgba="1.0 0.753 0.796 1" />
       </material>
     </visual>
@@ -72,5 +77,5 @@
         name="">
         <color
-          rgba="0.898039215686275 0.917647058823529 0.929411764705882 1" />
+          rgba="0.5 0.5 0.5 1" />
       </material>
     </visual>
@@ -125,5 +130,5 @@
         name="">
         <color
-          rgba="0.898039215686275 0.917647058823529 0.929411764705882 1" />
+          rgba="0.5 0.5 0.5 1" />
       </material>
     </visual>
@@ -178,5 +183,5 @@
         name="">
         <color
-          rgba="0.898039215686275 0.917647058823529 0.929411764705882 1" />
+          rgba="0.5 0.5 0.5 1" />
       </material>
     </visual>
@@ -231,5 +236,5 @@
         name="">
         <color
-          rgba="0.898039215686275 0.917647058823529 0.929411764705882 1" />
+          rgba="0.5 0.5 0.5 1" />
       </material>
     </visual>
@@ -269,5 +274,5 @@
             </geometry>
             <material name="">
-                <color rgba="1.0 0.0 0.0 1.0"/>
+                <color rgba="0.5373 0.8118 0.9412 1.0"/>
                 <texture filename=""/>
             </material>
@@ -281,5 +286,5 @@
     </link>
     <joint name="lidar_joint" type="fixed">
-        <origin xyz="0.04 0.0 0.045" rpy="1.5708 0.0 0.0"/>
+        <origin xyz="-0.03 0.0 0.045" rpy="1.5708 0.0 0.0"/>
         <parent link="base_link"/>
         <child link="lidar_link"/>
